File: Hardware/mood-badge.brd (EAGLE design)
At the start: 76.2 x 101.6 mm, 92 parts

Commit message: Updated BOM, minor tweaks to part values
Parts:
- C3, C5: value 0.1u -> 100n
- R26: value 100K -> 100k
- renumbered ARDUINO to MICROCONTROLLER
Changed lines of the file:
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@@
 </autorouter>
 <elements>
-<element name="ARDUINO" library="LinnesLab-Microcontrollers" package="TQFP32-08" package3d_urn="urn:adsk.eagle:package:18162361/2" value="ATMEGA328P_TQFP" x="52.324" y="73.66" smashed="yes" rot="MR0">
+<element name="MICROCONTROLLER" library="LinnesLab-Microcontrollers" package="TQFP32-08" package3d_urn="urn:adsk.eagle:package:18162361/2" value="ATMEGA328P_TQFP" x="52.324" y="73.66" smashed="yes" rot="MR0">
 <attribute name="NAME" x="52.324" y="67.691" size="0.7112" layer="26" ratio="20" rot="MR0" align="bottom-center"/>
 <attribute name="PROD_ID" value="IC-09069" x="52.324" y="73.66" size="1.778" layer="28" rot="MR0" display="off"/>
@@
 <attribute name="VALUE" x="60.071" y="68.199" size="1.27" layer="28" rot="MR0"/>
 </element>
-<element name="C3" library="LinnesLab-Passives" package="C0603" package3d_urn="urn:adsk.eagle:package:15661989/2" value="0.1u" x="60.96" y="75.184" smashed="yes" rot="MR90">
+<element name="C3" library="LinnesLab-Passives" package="C0603" package3d_urn="urn:adsk.eagle:package:15661989/2" value="100n" x="60.96" y="75.184" smashed="yes" rot="MR90">
 <attribute name="NAME" x="61.595" y="73.533" size="1.27" layer="26" rot="MR90"/>
 <attribute name="VALUE" x="61.595" y="76.073" size="1.27" layer="28" rot="MR90"/>
@@
 <attribute name="VALUE" x="49.403" y="82.169" size="1.27" layer="28" rot="MR90"/>
 </element>
-<element name="C5" library="LinnesLab-Passives" package="C0603" package3d_urn="urn:adsk.eagle:package:15661989/2" value="0.1u" x="52.832" y="81.28" smashed="yes" rot="MR270">
+<element name="C5" library="LinnesLab-Passives" package="C0603" package3d_urn="urn:adsk.eagle:package:15661989/2" value="100n" x="52.832" y="81.28" smashed="yes" rot="MR270">
 <attribute name="NAME" x="53.467" y="79.629" size="1.27" layer="26" rot="MR90"/>
 <attribute name="VALUE" x="53.467" y="82.169" size="1.27" layer="28" rot="MR90"/>
@@
 <attribute name="VALUE" x="15.875" y="41.783" size="0.7112" layer="28" rot="MR0"/>
 </element>
-<element name="R26" library="LinnesLab-Passives" package="R0603" package3d_urn="urn:adsk.eagle:package:15661944/2" value="100K" x="16.256" y="41.148" smashed="yes" rot="MR0">
+<element name="R26" library="LinnesLab-Passives" package="R0603" package3d_urn="urn:adsk.eagle:package:15661944/2" value="100k" x="16.256" y="41.148" smashed="yes" rot="MR0">
 <attribute name="NAME" x="17.907" y="39.751" size="0.7112" layer="26" rot="MR0"/>
 <attribute name="VALUE" x="15.875" y="39.751" size="0.7112" layer="28" rot="MR0"/>
@@
 <wire x1="10.16" y1="22.721" x2="12.966" y2="22.721" width="0.1524" layer="1"/>
 <wire x1="12.966" y1="22.721" x2="12.712" y2="21.9075" width="0.1524" layer="1"/>
-<contactref element="ARDUINO" pad="13"/>
+<contactref element="MICROCONTROLLER" pad="13"/>
 <wire x1="12.712" y1="13.6525" x2="12.712" y2="11.696" width="0.1524" layer="1"/>
 <wire x1="12.712" y1="11.696" x2="12.7" y2="11.684" width="0.1524" layer="1"/>
@@
 </signal>
 <signal name="SDA">
-<contactref element="ARDUINO" pad="27"/>
+<contactref element="MICROCONTROLLER" pad="27"/>
 </signal>
 <signal name="SCL">
-<contactref element="ARDUINO" pad="28"/>
+<contactref element="MICROCONTROLLER" pad="28"/>
 </signal>
 <signal name="RIGHT">
@@
 <wire x1="37.592" y1="22.721" x2="35.5995" y2="22.721" width="0.1524" layer="1"/>
 <wire x1="35.5995" y1="22.721" x2="35.04" y2="21.9075" width="0.1524" layer="1"/>
-<contactref element="ARDUINO" pad="11"/>
+<contactref element="MICROCONTROLLER" pad="11"/>
 <wire x1="35.04" y1="21.9075" x2="35.04" y2="23.864" width="0.1524" layer="1"/>
 <wire x1="35.04" y1="23.864" x2="35.052" y2="23.876" width="0.1524" layer="1"/>
@@
 </signal>
 <signal name="RXD">
-<contactref element="ARDUINO" pad="30"/>
+<contactref element="MICROCONTROLLER" pad="30"/>
 <contactref element="FTDI" pad="TXO"/>
 <wire x1="73.152" y1="85.09" x2="57.0267375" y2="85.09" width="0.1524" layer="16"/>
@@
 </signal>
 <signal name="TXD">
-<contactref element="ARDUINO" pad="31"/>
+<contactref element="MICROCONTROLLER" pad="31"/>
 <contactref element="FTDI" pad="RXI"/>
 <wire x1="73.152" y1="82.55" x2="56.134" y2="82.55" width="0.1524" layer="16"/>
@@
 <contactref element="R17" pad="2"/>
 <contactref element="MODE" pad="2"/>
-<contactref element="ARDUINO" pad="2"/>
+<contactref element="MICROCONTROLLER" pad="2"/>
 <contactref element="R16" pad="1"/>
 <via x="57.912" y="75.692" extent="1-16" drill="0.35"/>
@@
 </signal>
 <signal name="GND">
-<contactref element="ARDUINO" pad="21"/>
-<contactref element="ARDUINO" pad="3"/>
-<contactref element="ARDUINO" pad="5"/>
+<contactref element="MICROCONTROLLER" pad="21"/>
+<contactref element="MICROCONTROLLER" pad="3"/>
+<contactref element="MICROCONTROLLER" pad="5"/>
 <contactref element="C1" pad="2"/>
 <contactref element="C2" pad="2"/>
@@
 </signal>
 <signal name="N$1">
-<contactref element="ARDUINO" pad="7"/>
+<contactref element="MICROCONTROLLER" pad="7"/>
 <contactref element="C1" pad="1"/>
 <contactref element="XTAL" pad="1"/>
@@
 </signal>
 <signal name="VCC">
-<contactref element="ARDUINO" pad="18"/>
-<contactref element="ARDUINO" pad="4"/>
-<contactref element="ARDUINO" pad="6"/>
+<contactref element="MICROCONTROLLER" pad="18"/>
+<contactref element="MICROCONTROLLER" pad="4"/>
+<contactref element="MICROCONTROLLER" pad="6"/>
 <contactref element="C4" pad="1"/>
 <contactref element="C3" pad="1"/>
@@
 </signal>
 <signal name="N$2">
-<contactref element="ARDUINO" pad="8"/>
+<contactref element="MICROCONTROLLER" pad="8"/>
 <contactref element="C2" pad="1"/>
 <contactref element="XTAL" pad="2"/>
@@
 <contactref element="RESET" pad="4"/>
 <contactref element="RESET" pad="3"/>
-<contactref element="ARDUINO" pad="29"/>
+<contactref element="MICROCONTROLLER" pad="29"/>
 <contactref element="ICSP" pad="5"/>
 <contactref element="C5" pad="2"/>
@@
 <wire x1="28.5115" y1="31.408" x2="28.448" y2="31.408" width="0.1524" layer="1"/>
 <wire x1="28.448" y1="31.408" x2="25.908" y2="31.408" width="0.1524" layer="1"/>
-<contactref element="ARDUINO" pad="14"/>
+<contactref element="MICROCONTROLLER" pad="14"/>
 <wire x1="28.0035" y1="28.944" x2="29.96" y2="28.944" width="0.1524" layer="1"/>
 <wire x1="29.96" y1="28.944" x2="29.972" y2="28.956" width="0.1524" layer="1"/>
@@
 <wire x1="19.2405" y1="13.3105" x2="19.2405" y2="11.418" width="0.1524" layer="1"/>
 <wire x1="19.2405" y1="11.418" x2="19.7485" y2="10.656" width="0.1524" layer="1"/>
-<contactref element="ARDUINO" pad="12"/>
+<contactref element="MICROCONTROLLER" pad="12"/>
 <wire x1="28.0035" y1="10.656" x2="29.96" y2="10.656" width="0.1524" layer="1"/>
 <wire x1="29.96" y1="10.656" x2="29.972" y2="10.668" width="0.1524" layer="1"/>
@@
 <wire x1="54.356" y1="16.6885" x2="54.356" y2="18.962" width="0.1524" layer="1"/>
 <wire x1="54.356" y1="18.962" x2="51.816" y2="18.962" width="0.1524" layer="1"/>
-<contactref element="ARDUINO" pad="10"/>
+<contactref element="MICROCONTROLLER" pad="10"/>
 <wire x1="45.6565" y1="16.244" x2="45.6445" y2="16.256" width="0.1524" layer="1"/>
 <wire x1="45.6445" y1="16.256" x2="43.688" y2="16.256" width="0.1524" layer="1"/>
@@
 <wire x1="66.04" y1="23.8005" x2="65.5955" y2="23.356" width="0.1524" layer="1"/>
 <wire x1="66.04" y1="26.074" x2="63.5" y2="26.074" width="0.1524" layer="1"/>
-<contactref element="ARDUINO" pad="9"/>
+<contactref element="MICROCONTROLLER" pad="9"/>
 <wire x1="57.3405" y1="23.356" x2="55.384" y2="23.356" width="0.1524" layer="1"/>
 <wire x1="55.384" y1="23.356" x2="55.372" y2="23.368" width="0.1524" layer="1"/>
@@
 <wire x1="61.7054" y1="67.056" x2="63.5" y2="68.8506" width="0.1524" layer="16"/>
 <wire x1="63.5" y1="68.8506" x2="63.5" y2="75.692" width="0.1524" layer="16"/>
-<contactref element="ARDUINO" pad="26"/>
+<contactref element="MICROCONTROLLER" pad="26"/>
 <wire x1="50.7499125" y1="77.089" x2="50.616" y2="77.2229125" width="0.1524" layer="16"/>
 <wire x1="50.616" y1="77.2229125" x2="50.616" y2="77.6606" width="0.1524" layer="16"/>
@@
 <signal name="MISO">
 <contactref element="ICSP" pad="1"/>
-<contactref element="ARDUINO" pad="16"/>
+<contactref element="MICROCONTROLLER" pad="16"/>
 <wire x1="49.784" y1="71.12" x2="49.784" y2="69.6274" width="0.1524" layer="16"/>
 <wire x1="49.524" y1="69.3674" x2="49.784" y2="69.6274" width="0.1524" layer="16"/>
@@
 <signal name="SCK">
 <contactref element="ICSP" pad="3"/>
-<contactref element="ARDUINO" pad="17"/>
+<contactref element="MICROCONTROLLER" pad="17"/>
 <contactref element="RGB1" pad="CI_0"/>
 <wire x1="48.0314" y1="70.86" x2="48.2914" y2="71.12" width="0.1524" layer="16"/>
@@
 <signal name="MOSI">
 <contactref element="ICSP" pad="4"/>
-<contactref element="ARDUINO" pad="15"/>
+<contactref element="MICROCONTROLLER" pad="15"/>
 <contactref element="RGB1" pad="DI_0"/>
 <via x="50.8" y="71.12" extent="1-16" drill="0.35"/>
@@
 <signal name="SPKR">
 <contactref element="R29" pad="1"/>
-<contactref element="ARDUINO" pad="1"/>
+<contactref element="MICROCONTROLLER" pad="1"/>
 <wire x1="56.6166" y1="76.46" x2="49.2690875" y2="76.46" width="0.1524" layer="16"/>
 <wire x1="49.2690875" y1="76.46" x2="48.7610875" y2="76.968" width="0.1524" layer="16"/>

Commit message: Fixed diode numbering
Parts:
- renumbered D6 to D1
Changed lines of the file:
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@@
 <attribute name="VALUE" x="41.275" y="77.089" size="0.7112" layer="28" rot="MR90"/>
 </element>
-<element name="D6" library="LinnesLab-DiscreteSemi" package="USC" package3d_urn="urn:adsk.eagle:package:15664784/2" value="" x="38.1" y="73.66" smashed="yes" rot="MR180">
+<element name="D1" library="LinnesLab-DiscreteSemi" package="USC" package3d_urn="urn:adsk.eagle:package:15664784/2" value="" x="38.1" y="73.66" smashed="yes" rot="MR180">
 <attribute name="NAME" x="38.862" y="72.22" size="0.635" layer="26" rot="MR0"/>
 <attribute name="VALUE" x="36.83" y="75.325" size="0.635" layer="28" rot="MR180"/>
@@
 <wire x1="15.748" y1="45.212" x2="15.406" y2="45.55399375" width="0.6096" layer="16"/>
 <wire x1="15.406" y1="45.55399375" x2="15.406" y2="46.482" width="0.6096" layer="16"/>
-<contactref element="D6" pad="-"/>
+<contactref element="D1" pad="-"/>
 <contactref element="LS1" pad="+"/>
 <wire x1="10.16" y1="45.554" x2="13.025" y2="45.554" width="0.2032" layer="16"/>
@@
 <signal name="N$5">
 <contactref element="LS1" pad="-"/>
-<contactref element="D6" pad="+"/>
+<contactref element="D1" pad="+"/>
 <contactref element="Q1" pad="3"/>
 <wire x1="36.95" y1="73.66" x2="34.3" y2="73.66" width="0.1524" layer="16"/>
